Commit message: feat: Add robot enhancements

File: my_robot/urdf/my_robot.xacro (robot description, xacro)
@@ -54,3 +54,61 @@
     </visual>
   </link>
+  <joint type="continuous" name="left_wheel_hinge">
+    <origin xyz="0 0.15 0" rpy="0 0 0"/>
+    <child link="left_wheel"/>
+    <parent link="chassis"/>
+    <axis xyz="0 1 0" rpy="0 0 0"/>
+    <limit effort="10000" velocity="1000"/>
+    <dynamics damping="1.0" friction="1.0"/>
+  </joint>
+  <link name="left_wheel">
+    <inertial>
+      <mass value="5.0"/>
+      <origin xyz="0 0 0" rpy="0 0 0"/>
+      <inertia ixx="0.1" ixy="0" ixz="0"
+               iyy="0.1" iyz="0"
+               izz="0.1"/>
+    </inertial>
+    <collision name='left_wheel_collision'>
+      <origin xyz="0 -0.024 0" rpy=" 0 1.5707 1.5707"/>
+      <geometry>
+        <cylinder length="0.05" radius="0.0999"/>
+      </geometry>
+    </collision>
+    <visual name='left_wheel_visual'>
+      <origin xyz="0 -0.024 0" rpy=" 0 1.5707 1.5707"/>
+      <geometry>
+        <cylinder length="0.05" radius="0.1"/>
+      </geometry>
+    </visual>
+  </link>
+  <joint type="continuous" name="right_wheel_hinge">
+    <origin xyz="0 -0.15 0" rpy="0 0 0"/>
+    <child link="right_wheel"/>
+    <parent link="chassis"/>
+    <axis xyz="0 1 0" rpy="0 0 0"/>
+    <limit effort="10000" velocity="1000"/>
+    <dynamics damping="1.0" friction="1.0"/>
+  </joint>
+  <link name="right_wheel">
+    <inertial>
+      <mass value="5.0"/>
+      <origin xyz="0 0 0" rpy="0 0 0"/>
+      <inertia ixx="0.1" ixy="0" ixz="0"
+               iyy="0.1" iyz="0"
+               izz="0.1"/>
+    </inertial>
+    <collision name='right_wheel_collision'>
+      <origin xyz="0 0.024 0" rpy=" 0 1.5707 1.5707"/>
+      <geometry>
+        <cylinder length="0.05" radius="0.0999"/>
+      </geometry>
+    </collision>
+    <visual name='right_wheel_visual'>
+      <origin xyz="0 0.024 0" rpy=" 0 1.5707 1.5707"/>
+      <geometry>
+        <cylinder length="0.05" radius="0.1"/>
+      </geometry>
+    </visual>
+  </link>
 </robot>

Commit message: feat: Add camera and lidar links.

File: my_robot/urdf/my_robot.xacro (robot description, xacro)
@@ -112,3 +112,66 @@
     </visual>
   </link>
+  <joint type="fixed" name="camera_joint">
+    <origin xyz="0.2 0 0" rpy="0 0 0"/>
+    <child link="camera"/>
+    <parent link="chassis"/>
+    <axis xyz="0 1 0" rpy="0 0 0"/>
+  </joint>
+  <link name="camera">
+    <inertial>
+      <mass value="0.1"/>
+      <origin xyz="0.05 0.05 0.05" rpy="0 0 0"/>
+      <inertia ixx="1e-6" ixy="0" ixz="0"
+               iyy="1e-6" iyz="0"
+               izz="1e-6"/>
+    </inertial>
+    <collision name='camera_collision'>
+      <origin xyz="0 0 0" rpy=" 0 0 0"/>
+      <geometry>
+        <box size="0.05 0.05 0.05"/>
+      </geometry>
+    </collision>
+    <visual name='camera_visual'>
+      <origin xyz="0 0 0" rpy=" 0 0 0"/>
+      <geometry>
+        <box size="0.05 0.05 0.05"/>
+      </geometry>
+    </visual>
+  </link>
+  <joint type="fixed" name="hokuyo_joint">
+    <origin xyz="0.15 0 0.1" rpy="0 0 0"/>
+    <child link="hokuyo"/>
+    <parent link="chassis"/>
+    <axis xyz="0 1 0" rpy="0 0 0"/>
+  </joint>
+  <link name="hokuyo">
+    <inertial>
+      <mass value="1e-5"/>
+      <origin xyz="0 0 0" rpy="0 0 0"/>
+      <inertia ixx="1e-6" ixy="0" ixz="0"
+               iyy="1e-6" iyz="0"
+               izz="1e-6"/>
+    </inertial>
+    <collision name='hokuyo_collision'>
+      <origin xyz="0 0 0" rpy=" 0 0 0"/>
+      <geometry>
+        <box size="0.1 0.1 0.1"/>
+      </geometry>
+    </collision>
+    <visual name='hokuyo_visual'>
+      <origin xyz="0 0 0" rpy=" 0 0 0"/>
+      <geometry>
+        <mesh filename="package://my_robot/meshes/hokuyo.dae"/>
+      </geometry>
+    </visual>
+  </link>
+<gazebo reference="left_wheel">
+    <material>Gazebo/Green</material>
+</gazebo>
+<gazebo reference="right_wheel">
+    <material>Gazebo/Green</material>
+</gazebo>
+<gazebo reference="chassis">
+    <material>Gazebo/Red</material>
+</gazebo>
 </robot>

Commit message: fix: Camera and laser plugins tested and fixed.

File: my_robot/urdf/my_robot.xacro (robot description, xacro)
@@ -1,6 +1,7 @@
 <?xml version='1.0'?>
 <robot name="my_robot" xmlns:xacro="http://www.ros.org/wiki/xacro">
+  <xacro:include filename="$(find my_robot)/urdf/my_robot.gazebo"/>
   <link name="robot_footprint"></link>
-  <joint name="robot_foorprint_joint" type="fixed">
+  <joint name="robot_footprint_joint" type="fixed">
     <origin xyz="0 0 0" rpy="0 0 0"/>
     <parent link="robot_footprint"/>
@@ -8,5 +9,5 @@
   </joint>
   <link name='chassis'>
-    <pose>0 0 0.1 0 0 0</pose>
+    <origin xyz="0 0 0" rpy="0 0 0"/>
     <inertial>
       <mass value="15.0"/>
@@ -17,5 +18,5 @@
       />
     </inertial>
-    <collision name='collision'>
+    <collision name='chassis_collision'>
       <origin xyz="0 0 0" rpy=" 0 0 0"/>
       <geometry>
@@ -63,7 +64,7 @@
   </joint>
   <link name="left_wheel">
+    <origin xyz="0 0 0" rpy="0 0 0"/>
     <inertial>
       <mass value="5.0"/>
-      <origin xyz="0 0 0" rpy="0 0 0"/>
       <inertia ixx="0.1" ixy="0" ixz="0"
                iyy="0.1" iyz="0"
@@ -71,11 +72,11 @@
     </inertial>
     <collision name='left_wheel_collision'>
-      <origin xyz="0 -0.024 0" rpy=" 0 1.5707 1.5707"/>
+      <origin xyz="0 0 0" rpy=" 0 1.5707 1.5707"/>
       <geometry>
-        <cylinder length="0.05" radius="0.0999"/>
+        <cylinder length="0.05" radius="0.1"/>
       </geometry>
     </collision>
     <visual name='left_wheel_visual'>
-      <origin xyz="0 -0.024 0" rpy=" 0 1.5707 1.5707"/>
+      <origin xyz="0 0 0" rpy=" 0 1.5707 1.5707"/>
       <geometry>
         <cylinder length="0.05" radius="0.1"/>
@@ -92,7 +93,7 @@
   </joint>
   <link name="right_wheel">
+    <origin xyz="0 0 0" rpy="0 0 0"/>
     <inertial>
       <mass value="5.0"/>
-      <origin xyz="0 0 0" rpy="0 0 0"/>
       <inertia ixx="0.1" ixy="0" ixz="0"
                iyy="0.1" iyz="0"
@@ -100,11 +101,11 @@
     </inertial>
     <collision name='right_wheel_collision'>
-      <origin xyz="0 0.024 0" rpy=" 0 1.5707 1.5707"/>
+      <origin xyz="0 0 0" rpy=" 0 1.5707 1.5707"/>
       <geometry>
-        <cylinder length="0.05" radius="0.0999"/>
+        <cylinder length="0.05" radius="0.1"/>
       </geometry>
     </collision>
     <visual name='right_wheel_visual'>
-      <origin xyz="0 0.024 0" rpy=" 0 1.5707 1.5707"/>
+      <origin xyz="0 0 0" rpy=" 0 1.5707 1.5707"/>
       <geometry>
         <cylinder length="0.05" radius="0.1"/>
@@ -119,7 +120,7 @@
   </joint>
   <link name="camera">
+    <origin xyz="0 0 0" rpy="0 0 0"/>
     <inertial>
       <mass value="0.1"/>
-      <origin xyz="0.05 0.05 0.05" rpy="0 0 0"/>
       <inertia ixx="1e-6" ixy="0" ixz="0"
                iyy="1e-6" iyz="0"
@@ -146,7 +147,7 @@
   </joint>
   <link name="hokuyo">
+    <origin xyz="0 0 0" rpy="0 0 0"/>
     <inertial>
       <mass value="1e-5"/>
-      <origin xyz="0 0 0" rpy="0 0 0"/>
       <inertia ixx="1e-6" ixy="0" ixz="0"
                iyy="1e-6" iyz="0"

Commit message: feat: Add skid-steer robot

File: my_robot/urdf/my_robot.xacro (robot description, xacro)
@@ -11,5 +11,5 @@
     <origin xyz="0 0 0" rpy="0 0 0"/>
     <inertial>
-      <mass value="15.0"/>
+      <mass value="20.0"/>
       <origin xyz="0 0 0" rpy="0 0 0"/>
       <inertia ixx="0.1" ixy="0" ixz="0"
@@ -21,5 +21,5 @@
       <origin xyz="0 0 0" rpy=" 0 0 0"/>
       <geometry>
-        <box size=".4 .2 .1"/>
+        <box size=".6 .3 .1"/>
       </geometry>
     </collision>
@@ -27,84 +27,130 @@
       <origin xyz="0 0 0" rpy=" 0 0 0"/>
       <geometry>
-        <box size=".4 .2 .1"/>
-      </geometry>
-    </visual>
-    <collision name='back_caster_collision'>
-      <origin xyz="-0.15 0 -0.05" rpy=" 0 0 0"/>
-      <geometry>
-        <sphere radius="0.0499"/>
-      </geometry>
-    </collision>
-    <visual name='back_caster_visual'>
-      <origin xyz="-0.15 0 -0.05" rpy=" 0 0 0"/>
-      <geometry>
-        <sphere radius="0.05"/>
-      </geometry>
-    </visual>
-    <collision name='front_caster_collision'>
-      <origin xyz="0.15 0 -0.05" rpy=" 0 0 0"/>
-      <geometry>
-        <sphere radius="0.0499"/>
-      </geometry>
-    </collision>
-    <visual name='front_caster_visual'>
-      <origin xyz="0.15 0 -0.05" rpy=" 0 0 0"/>
-      <geometry>
-        <sphere radius="0.05"/>
-      </geometry>
-    </visual>
-  </link>
-  <joint type="continuous" name="left_wheel_hinge">
-    <origin xyz="0 0.15 0" rpy="0 0 0"/>
-    <child link="left_wheel"/>
-    <parent link="chassis"/>
-    <axis xyz="0 1 0" rpy="0 0 0"/>
-    <limit effort="10000" velocity="1000"/>
-    <dynamics damping="1.0" friction="1.0"/>
-  </joint>
-  <link name="left_wheel">
-    <origin xyz="0 0 0" rpy="0 0 0"/>
-    <inertial>
-      <mass value="5.0"/>
-      <inertia ixx="0.1" ixy="0" ixz="0"
-               iyy="0.1" iyz="0"
-               izz="0.1"/>
-    </inertial>
-    <collision name='left_wheel_collision'>
-      <origin xyz="0 0 0" rpy=" 0 1.5707 1.5707"/>
-      <geometry>
-        <cylinder length="0.05" radius="0.1"/>
-      </geometry>
-    </collision>
-    <visual name='left_wheel_visual'>
-      <origin xyz="0 0 0" rpy=" 0 1.5707 1.5707"/>
-      <geometry>
-        <cylinder length="0.05" radius="0.1"/>
-      </geometry>
-    </visual>
-  </link>
-  <joint type="continuous" name="right_wheel_hinge">
-    <origin xyz="0 -0.15 0" rpy="0 0 0"/>
-    <child link="right_wheel"/>
-    <parent link="chassis"/>
-    <axis xyz="0 1 0" rpy="0 0 0"/>
-    <limit effort="10000" velocity="1000"/>
-    <dynamics damping="1.0" friction="1.0"/>
-  </joint>
-  <link name="right_wheel">
-    <origin xyz="0 0 0" rpy="0 0 0"/>
-    <inertial>
-      <mass value="5.0"/>
-      <inertia ixx="0.1" ixy="0" ixz="0"
-               iyy="0.1" iyz="0"
-               izz="0.1"/>
-    </inertial>
-    <collision name='right_wheel_collision'>
-      <origin xyz="0 0 0" rpy=" 0 1.5707 1.5707"/>
-      <geometry>
-        <cylinder length="0.05" radius="0.1"/>
-      </geometry>
-    </collision>
-    <visual name='right_wheel_visual'>
+        <box size=".6 .3 .15"/>
+      </geometry>
+    </visual>
+    <collision name='hokuyo_base_collision'>
+      <origin xyz="0 0 0.12" rpy=" 0 0 0"/>
+      <geometry>
+        <cylinder length="0.1" radius="0.05"/>
+      </geometry>
+    </collision>
+    <visual name='hokuyo_base_visual'>
+      <origin xyz="0 0 0.12" rpy=" 0 0 0"/>
+      <geometry>
+        <cylinder length="0.1" radius="0.05"/>
+      </geometry>
+    </visual>
+  </link>
+  <joint type="continuous" name="front_left_wheel_hinge">
+    <origin xyz="0.25 0.2 0" rpy="0 0 0"/>
+    <child link="front_left_wheel"/>
+    <parent link="chassis"/>
+    <axis xyz="0 1 0" rpy="0 0 0"/>
+    <limit effort="10000" velocity="1000"/>
+    <dynamics damping="1.0" friction="1.0"/>
+  </joint>
+  <link name="front_left_wheel">
+    <origin xyz="0 0 0" rpy="0 0 0"/>
+    <inertial>
+      <mass value="5.0"/>
+      <inertia ixx="0.1" ixy="0" ixz="0"
+               iyy="0.1" iyz="0"
+               izz="0.1"/>
+    </inertial>
+    <collision name='front_left_wheel_collision'>
+      <origin xyz="0 0 0" rpy=" 0 1.5707 1.5707"/>
+      <geometry>
+        <cylinder length="0.05" radius="0.1"/>
+      </geometry>
+    </collision>
+    <visual name='front_left_wheel_visual'>
+      <origin xyz="0 0 0" rpy=" 0 1.5707 1.5707"/>
+      <geometry>
+        <cylinder length="0.05" radius="0.1"/>
+      </geometry>
+    </visual>
+  </link>
+  <joint type="continuous" name="front_right_wheel_hinge">
+    <origin xyz="0.25 -0.2 0" rpy="0 0 0"/>
+    <child link="front_right_wheel"/>
+    <parent link="chassis"/>
+    <axis xyz="0 1 0" rpy="0 0 0"/>
+    <limit effort="10000" velocity="1000"/>
+    <dynamics damping="1.0" friction="1.0"/>
+  </joint>
+  <link name="front_right_wheel">
+    <origin xyz="0 0 0" rpy="0 0 0"/>
+    <inertial>
+      <mass value="5.0"/>
+      <inertia ixx="0.1" ixy="0" ixz="0"
+               iyy="0.1" iyz="0"
+               izz="0.1"/>
+    </inertial>
+    <collision name='front_right_wheel_collision'>
+      <origin xyz="0 0 0" rpy=" 0 1.5707 1.5707"/>
+      <geometry>
+        <cylinder length="0.05" radius="0.1"/>
+      </geometry>
+    </collision>
+    <visual name='front_right_wheel_visual'>
+      <origin xyz="0 0 0" rpy=" 0 1.5707 1.5707"/>
+      <geometry>
+        <cylinder length="0.05" radius="0.1"/>
+      </geometry>
+    </visual>
+  </link>
+  <joint type="continuous" name="back_left_wheel_hinge">
+    <origin xyz="-0.25 0.2 0" rpy="0 0 0"/>
+    <child link="back_left_wheel"/>
+    <parent link="chassis"/>
+    <axis xyz="0 1 0" rpy="0 0 0"/>
+    <limit effort="10000" velocity="1000"/>
+    <dynamics damping="1.0" friction="1.0"/>
+  </joint>
+  <link name="back_left_wheel">
+    <origin xyz="0 0 0" rpy="0 0 0"/>
+    <inertial>
+      <mass value="5.0"/>
+      <inertia ixx="0.1" ixy="0" ixz="0"
+               iyy="0.1" iyz="0"
+               izz="0.1"/>
+    </inertial>
+    <collision name='back_left_wheel_collision'>
+      <origin xyz="0 0 0" rpy=" 0 1.5707 1.5707"/>
+      <geometry>
+        <cylinder length="0.05" radius="0.1"/>
+      </geometry>
+    </collision>
+    <visual name='back_left_wheel_visual'>
+      <origin xyz="0 0 0" rpy=" 0 1.5707 1.5707"/>
+      <geometry>
+        <cylinder length="0.05" radius="0.1"/>
+      </geometry>
+    </visual>
+  </link>
+  <joint type="continuous" name="back_right_wheel_hinge">
+    <origin xyz="-0.25 -0.2 0" rpy="0 0 0"/>
+    <child link="back_right_wheel"/>
+    <parent link="chassis"/>
+    <axis xyz="0 1 0" rpy="0 0 0"/>
+    <limit effort="10000" velocity="1000"/>
+    <dynamics damping="1.0" friction="1.0"/>
+  </joint>
+  <link name="back_right_wheel">
+    <origin xyz="0 0 0" rpy="0 0 0"/>
+    <inertial>
+      <mass value="5.0"/>
+      <inertia ixx="0.1" ixy="0" ixz="0"
+               iyy="0.1" iyz="0"
+               izz="0.1"/>
+    </inertial>
+    <collision name='back_right_wheel_collision'>
+      <origin xyz="0 0 0" rpy=" 0 1.5707 1.5707"/>
+      <geometry>
+        <cylinder length="0.05" radius="0.1"/>
+      </geometry>
+    </collision>
+    <visual name='back_right_wheel_visual'>
       <origin xyz="0 0 0" rpy=" 0 1.5707 1.5707"/>
       <geometry>
@@ -114,5 +160,5 @@
   </link>
   <joint type="fixed" name="camera_joint">
-    <origin xyz="0.2 0 0" rpy="0 0 0"/>
+    <origin xyz="0.3 0 0.04" rpy="0 0 0"/>
     <child link="camera"/>
     <parent link="chassis"/>
@@ -141,5 +187,5 @@
   </link>
   <joint type="fixed" name="hokuyo_joint">
-    <origin xyz="0.15 0 0.1" rpy="0 0 0"/>
+    <origin xyz="0 0 0.2" rpy="0 0 0"/>
     <child link="hokuyo"/>
     <parent link="chassis"/>
@@ -167,12 +213,21 @@
     </visual>
   </link>
-<gazebo reference="left_wheel">
+<gazebo reference="front_left_wheel">
+    <material>Gazebo/Black</material>
+</gazebo>
+<gazebo reference="front_right_wheel">
+    <material>Gazebo/Black</material>
+</gazebo>
+<gazebo reference="back_left_wheel">
+    <material>Gazebo/Black</material>
+</gazebo>
+<gazebo reference="back_right_wheel">
+    <material>Gazebo/Black</material>
+</gazebo>
+<gazebo reference="chassis">
+    <material>Gazebo/Purple</material>
+</gazebo>
+<gazebo reference="camera">
     <material>Gazebo/Green</material>
 </gazebo>
-<gazebo reference="right_wheel">
-    <material>Gazebo/Green</material>
-</gazebo>
-<gazebo reference="chassis">
-    <material>Gazebo/Red</material>
-</gazebo>
 </robot>

Commit message: feat: Add rtab-map to map the world

File: my_robot/urdf/my_robot.xacro (robot description, xacro)
@@ -161,9 +161,9 @@
   <joint type="fixed" name="camera_joint">
     <origin xyz="0.3 0 0.04" rpy="0 0 0"/>
-    <child link="camera"/>
-    <parent link="chassis"/>
-    <axis xyz="0 1 0" rpy="0 0 0"/>
-  </joint>
-  <link name="camera">
+    <child link="camera_link"/>
+    <parent link="chassis"/>
+    <axis xyz="0 1 0" rpy="0 0 0"/>
+  </joint>
+  <link name="camera_link">
     <origin xyz="0 0 0" rpy="0 0 0"/>
     <inertial>
@@ -186,4 +186,11 @@
     </visual>
   </link>
+  <joint type="fixed" name="camera_optical_joint">
+    <origin xyz="0 0 0" rpy="-1.5707 0 -1.5707"/>
+    <parent link="camera_link"/>
+    <child link="camera_link_optical"/>
+  </joint>
+  <link name="camera_link_optical">
+  </link>
   <joint type="fixed" name="hokuyo_joint">
     <origin xyz="0 0 0.2" rpy="0 0 0"/>
